File: KarisGiftPCB/KarisGiftPCB.sch (KiCad schematic (older format))
At the start: 43 parts, among them J1 Conn_01x03_Female, J2 Conn_02x03_Top_Bottom, J3 Conn_01x02_Female, J4 Conn_02x20_Top_Bottom, J5 Conn_01x02_Female, Q1 2N3904, Q2 2N3906, Q3 2N3904, Q4 2N3904, Q5 2N3904, U1 ATtiny85V-10PU

Commit message: Made new Kicad project for PCB schematic and layout. Started layout.
Parts:
- D1: footprint Diode_THT:D_5W_P12.70mm_Horizontal -> Diode_THT:D_DO-41_SOD81_P10.16mm_Horizontal
- J1: footprint (none) -> Connector_PinSocket_2.54mm:PinSocket_1x03_P2.54mm_Vertical
- J2: footprint (none) -> Connector_PinSocket_2.54mm:PinSocket_2x03_P2.54mm_Vertical
- J3, J5: footprint (none) -> Connector_PinSocket_2.54mm:PinSocket_1x02_P2.54mm_Vertical
- J4: footprint (none) -> Connector_PinSocket_2.54mm:PinSocket_2x20_P2.54mm_Vertical
- R1, R10, R11, R12, R13, R14, R15, R16, R17, R18, R19, R2, R20, R21, R22, R23, R24, R25, R26, R27, R28, R29, R3, R30, R31, R4, R5, R6, R7, R8, R9: footprint (none) -> Resistor_THT:R_Axial_DIN0207_L6.3mm_D2.5mm_P10.16mm_Horizontal
- U1: symbol KarisGift-rescue:ATtiny85V-10PU-MCU_Microchip_ATtiny -> KarisGiftPCB-rescue:ATtiny85V-10PU-MCU_Microchip_ATtiny-KarisGift-rescue-KarisGiftPCB-rescue
Changed lines of the file:
@@
 $EndDescr
 $Comp
-L KarisGift-rescue:ATtiny85V-10PU-MCU_Microchip_ATtiny U1
+L KarisGiftPCB-rescue:ATtiny85V-10PU-MCU_Microchip_ATtiny-KarisGift-rescue-KarisGiftPCB-rescue U1
 U 1 1 5FDE0C7F
 P 1900 1700
@@
 F 0 "R6" H 5220 1946 50  0000 L CNN
 F 1 "R" H 5220 1855 50  0000 L CNN
-F 2 "" V 5080 1900 50  0001 C CNN
+F 2 "Resistor_THT:R_Axial_DIN0207_L6.3mm_D2.5mm_P10.16mm_Horizontal" V 5080 1900 50  0001 C CNN
 F 3 "~" H 5150 1900 50  0001 C CNN
 	1    5150 1900
@@
 F 0 "R19" H 6320 1946 50  0000 L CNN
 F 1 "R" H 6320 1855 50  0000 L CNN
-F 2 "" V 6180 1900 50  0001 C CNN
+F 2 "Resistor_THT:R_Axial_DIN0207_L6.3mm_D2.5mm_P10.16mm_Horizontal" V 6180 1900 50  0001 C CNN
 F 3 "~" H 6250 1900 50  0001 C CNN
 	1    6250 1900
@@
 F 0 "R8" V 5200 2450 50  0000 C CNN
 F 1 "500" V 5300 2500 50  0000 C CNN
-F 2 "" V 5230 2500 50  0001 C CNN
+F 2 "Resistor_THT:R_Axial_DIN0207_L6.3mm_D2.5mm_P10.16mm_Horizontal" V 5230 2500 50  0001 C CNN
 F 3 "~" H 5300 2500 50  0001 C CNN
 	1    5300 2500
@@
 F 0 "R30" V 8150 1900 50  0000 C CNN
 F 1 "500" V 8250 1950 50  0000 C CNN
-F 2 "" V 8180 1950 50  0001 C CNN
+F 2 "Resistor_THT:R_Axial_DIN0207_L6.3mm_D2.5mm_P10.16mm_Horizontal" V 8180 1950 50  0001 C CNN
 F 3 "~" H 8250 1950 50  0001 C CNN
 	1    8250 1950
@@
 F 0 "D1" V 8304 1480 50  0000 L CNN
 F 1 "D" V 8395 1480 50  0000 L CNN
-F 2 "Diode_THT:D_5W_P12.70mm_Horizontal" H 8350 1400 50  0001 C CNN
+F 2 "Diode_THT:D_DO-41_SOD81_P10.16mm_Horizontal" H 8350 1400 50  0001 C CNN
 F 3 "~" H 8350 1400 50  0001 C CNN
 	1    8350 1400
@@
 F 0 "R31" H 8250 1950 50  0000 L CNN
 F 1 "10k" V 8400 2050 50  0000 L CNN
-F 2 "" V 8330 2100 50  0001 C CNN
+F 2 "Resistor_THT:R_Axial_DIN0207_L6.3mm_D2.5mm_P10.16mm_Horizontal" V 8330 2100 50  0001 C CNN
 F 3 "~" H 8400 2100 50  0001 C CNN
 	1    8400 2100
@@
 F 0 "R1" V 1250 3950 50  0000 C CNN
 F 1 "500" V 1350 4000 50  0000 C CNN
-F 2 "" V 1280 4000 50  0001 C CNN
+F 2 "Resistor_THT:R_Axial_DIN0207_L6.3mm_D2.5mm_P10.16mm_Horizontal" V 1280 4000 50  0001 C CNN
 F 3 "~" H 1350 4000 50  0001 C CNN
 	1    1350 4000
@@
 F 0 "R3" V 1600 5100 50  0000 C CNN
 F 1 "470" V 1500 5050 50  0000 C CNN
-F 2 "" V 1430 5050 50  0001 C CNN
+F 2 "Resistor_THT:R_Axial_DIN0207_L6.3mm_D2.5mm_P10.16mm_Horizontal" V 1430 5050 50  0001 C CNN
 F 3 "~" H 1500 5050 50  0001 C CNN
 	1    1500 5050
@@
 F 0 "R5" H 2200 3750 50  0000 C CNN
 F 1 "10k" V 2300 3600 50  0000 C CNN
-F 2 "" V 2230 3600 50  0001 C CNN
+F 2 "Resistor_THT:R_Axial_DIN0207_L6.3mm_D2.5mm_P10.16mm_Horizontal" V 2230 3600 50  0001 C CNN
 F 3 "~" H 2300 3600 50  0001 C CNN
 	1    2300 3600
@@
 F 0 "R4" V 1950 3700 50  0000 C CNN
 F 1 "500" V 2050 3800 50  0000 C CNN
-F 2 "" V 1980 3800 50  0001 C CNN
+F 2 "Resistor_THT:R_Axial_DIN0207_L6.3mm_D2.5mm_P10.16mm_Horizontal" V 1980 3800 50  0001 C CNN
 F 3 "~" H 2050 3800 50  0001 C CNN
 	1    2050 3800
@@
 F 0 "R2" H 1400 4000 50  0000 C CNN
 F 1 "10k" V 1500 4150 50  0000 C CNN
-F 2 "" V 1430 4150 50  0001 C CNN
+F 2 "Resistor_THT:R_Axial_DIN0207_L6.3mm_D2.5mm_P10.16mm_Horizontal" V 1430 4150 50  0001 C CNN
 F 3 "~" H 1500 4150 50  0001 C CNN
 	1    1500 4150
@@
 F 0 "R11" H 5300 2500 50  0000 L CNN
 F 1 "10k" V 5450 2600 50  0000 L CNN
-F 2 "" V 5380 2650 50  0001 C CNN
+F 2 "Resistor_THT:R_Axial_DIN0207_L6.3mm_D2.5mm_P10.16mm_Horizontal" V 5380 2650 50  0001 C CNN
 F 3 "~" H 5450 2650 50  0001 C CNN
 	1    5450 2650
@@
 F 0 "J1" H 3128 5076 50  0000 L CNN
 F 1 "Conn_01x03_Female" H 2300 5300 50  0000 L CNN
-F 2 "" H 3100 5050 50  0001 C CNN
+F 2 "Connector_PinSocket_2.54mm:PinSocket_1x03_P2.54mm_Vertical" H 3100 5050 50  0001 C CNN
 F 3 "~" H 3100 5050 50  0001 C CNN
 	1    3100 5050
@@
 F 0 "J5" H 8928 1326 50  0000 L CNN
 F 1 "Conn_01x02_Female" H 8500 1150 50  0000 L CNN
-F 2 "" H 8900 1350 50  0001 C CNN
+F 2 "Connector_PinSocket_2.54mm:PinSocket_1x02_P2.54mm_Vertical" H 8900 1350 50  0001 C CNN
 F 3 "~" H 8900 1350 50  0001 C CNN
 	1    8900 1350
@@
 F 0 "J4" V 6146 2430 50  0000 L CNN
 F 1 "Conn_02x20_Top_Bottom" V 6450 950 50  0000 L CNN
-F 2 "" H 6050 1450 50  0001 C CNN
+F 2 "Connector_PinSocket_2.54mm:PinSocket_2x20_P2.54mm_Vertical" H 6050 1450 50  0001 C CNN
 F 3 "~" H 6050 1450 50  0001 C CNN
 	1    6050 1450
@@
 F 0 "R7" H 5320 1946 50  0000 L CNN
 F 1 "R" H 5320 1855 50  0000 L CNN
-F 2 "" V 5180 1900 50  0001 C CNN
+F 2 "Resistor_THT:R_Axial_DIN0207_L6.3mm_D2.5mm_P10.16mm_Horizontal" V 5180 1900 50  0001 C CNN
 F 3 "~" H 5250 1900 50  0001 C CNN
 	1    5250 1900
@@
 F 0 "R9" H 5420 1946 50  0000 L CNN
 F 1 "R" H 5420 1855 50  0000 L CNN
-F 2 "" V 5280 1900 50  0001 C CNN
+F 2 "Resistor_THT:R_Axial_DIN0207_L6.3mm_D2.5mm_P10.16mm_Horizontal" V 5280 1900 50  0001 C CNN
 F 3 "~" H 5350 1900 50  0001 C CNN
 	1    5350 1900
@@
 F 0 "R10" H 5520 1946 50  0000 L CNN
 F 1 "R" H 5520 1855 50  0000 L CNN
-F 2 "" V 5380 1900 50  0001 C CNN
+F 2 "Resistor_THT:R_Axial_DIN0207_L6.3mm_D2.5mm_P10.16mm_Horizontal" V 5380 1900 50  0001 C CNN
 F 3 "~" H 5450 1900 50  0001 C CNN
 	1    5450 1900
@@
 F 0 "R12" H 5620 1946 50  0000 L CNN
 F 1 "R" H 5620 1855 50  0000 L CNN
-F 2 "" V 5480 1900 50  0001 C CNN
+F 2 "Resistor_THT:R_Axial_DIN0207_L6.3mm_D2.5mm_P10.16mm_Horizontal" V 5480 1900 50  0001 C CNN
 F 3 "~" H 5550 1900 50  0001 C CNN
 	1    5550 1900
@@
 F 0 "R13" H 5720 1946 50  0000 L CNN
 F 1 "R" H 5720 1855 50  0000 L CNN
-F 2 "" V 5580 1900 50  0001 C CNN
+F 2 "Resistor_THT:R_Axial_DIN0207_L6.3mm_D2.5mm_P10.16mm_Horizontal" V 5580 1900 50  0001 C CNN
 F 3 "~" H 5650 1900 50  0001 C CNN
 	1    5650 1900
@@
 F 0 "R14" H 5820 1946 50  0000 L CNN
 F 1 "R" H 5820 1855 50  0000 L CNN
-F 2 "" V 5680 1900 50  0001 C CNN
+F 2 "Resistor_THT:R_Axial_DIN0207_L6.3mm_D2.5mm_P10.16mm_Horizontal" V 5680 1900 50  0001 C CNN
 F 3 "~" H 5750 1900 50  0001 C CNN
 	1    5750 1900
@@
 F 0 "R15" H 5920 1946 50  0000 L CNN
 F 1 "R" H 5920 1855 50  0000 L CNN
-F 2 "" V 5780 1900 50  0001 C CNN
+F 2 "Resistor_THT:R_Axial_DIN0207_L6.3mm_D2.5mm_P10.16mm_Horizontal" V 5780 1900 50  0001 C CNN
 F 3 "~" H 5850 1900 50  0001 C CNN
 	1    5850 1900
@@
 F 0 "R16" H 6020 1946 50  0000 L CNN
 F 1 "R" H 6020 1855 50  0000 L CNN
-F 2 "" V 5880 1900 50  0001 C CNN
+F 2 "Resistor_THT:R_Axial_DIN0207_L6.3mm_D2.5mm_P10.16mm_Horizontal" V 5880 1900 50  0001 C CNN
 F 3 "~" H 5950 1900 50  0001 C CNN
 	1    5950 1900
@@
 F 0 "R17" H 6120 1946 50  0000 L CNN
 F 1 "R" H 6120 1855 50  0000 L CNN
-F 2 "" V 5980 1900 50  0001 C CNN
+F 2 "Resistor_THT:R_Axial_DIN0207_L6.3mm_D2.5mm_P10.16mm_Horizontal" V 5980 1900 50  0001 C CNN
 F 3 "~" H 6050 1900 50  0001 C CNN
 	1    6050 1900
@@
 F 0 "R18" H 6220 1946 50  0000 L CNN
 F 1 "R" H 6220 1855 50  0000 L CNN
-F 2 "" V 6080 1900 50  0001 C CNN
+F 2 "Resistor_THT:R_Axial_DIN0207_L6.3mm_D2.5mm_P10.16mm_Horizontal" V 6080 1900 50  0001 C CNN
 F 3 "~" H 6150 1900 50  0001 C CNN
 	1    6150 1900
@@
 F 0 "R20" H 6420 1946 50  0000 L CNN
 F 1 "R" H 6420 1855 50  0000 L CNN
-F 2 "" V 6280 1900 50  0001 C CNN
+F 2 "Resistor_THT:R_Axial_DIN0207_L6.3mm_D2.5mm_P10.16mm_Horizontal" V 6280 1900 50  0001 C CNN
 F 3 "~" H 6350 1900 50  0001 C CNN
 	1    6350 1900
@@
 F 0 "R21" H 6520 1946 50  0000 L CNN
 F 1 "R" H 6520 1855 50  0000 L CNN
-F 2 "" V 6380 1900 50  0001 C CNN
+F 2 "Resistor_THT:R_Axial_DIN0207_L6.3mm_D2.5mm_P10.16mm_Horizontal" V 6380 1900 50  0001 C CNN
 F 3 "~" H 6450 1900 50  0001 C CNN
 	1    6450 1900
@@
 F 0 "R23" H 6620 1946 50  0000 L CNN
 F 1 "R" H 6620 1855 50  0000 L CNN
-F 2 "" V 6480 1900 50  0001 C CNN
+F 2 "Resistor_THT:R_Axial_DIN0207_L6.3mm_D2.5mm_P10.16mm_Horizontal" V 6480 1900 50  0001 C CNN
 F 3 "~" H 6550 1900 50  0001 C CNN
 	1    6550 1900
@@
 F 0 "R25" H 6720 1946 50  0000 L CNN
 F 1 "R" H 6720 1855 50  0000 L CNN
-F 2 "" V 6580 1900 50  0001 C CNN
+F 2 "Resistor_THT:R_Axial_DIN0207_L6.3mm_D2.5mm_P10.16mm_Horizontal" V 6580 1900 50  0001 C CNN
 F 3 "~" H 6650 1900 50  0001 C CNN
 	1    6650 1900
@@
 F 0 "R26" H 6820 1946 50  0000 L CNN
 F 1 "R" H 6820 1855 50  0000 L CNN
-F 2 "" V 6680 1900 50  0001 C CNN
+F 2 "Resistor_THT:R_Axial_DIN0207_L6.3mm_D2.5mm_P10.16mm_Horizontal" V 6680 1900 50  0001 C CNN
 F 3 "~" H 6750 1900 50  0001 C CNN
 	1    6750 1900
@@
 F 0 "R27" H 6920 1946 50  0000 L CNN
 F 1 "R" H 6920 1855 50  0000 L CNN
-F 2 "" V 6780 1900 50  0001 C CNN
+F 2 "Resistor_THT:R_Axial_DIN0207_L6.3mm_D2.5mm_P10.16mm_Horizontal" V 6780 1900 50  0001 C CNN
 F 3 "~" H 6850 1900 50  0001 C CNN
 	1    6850 1900
@@
 F 0 "R28" H 7020 1946 50  0000 L CNN
 F 1 "R" H 7020 1855 50  0000 L CNN
-F 2 "" V 6880 1900 50  0001 C CNN
+F 2 "Resistor_THT:R_Axial_DIN0207_L6.3mm_D2.5mm_P10.16mm_Horizontal" V 6880 1900 50  0001 C CNN
 F 3 "~" H 6950 1900 50  0001 C CNN
 	1    6950 1900
@@
 F 0 "R29" H 7120 1946 50  0000 L CNN
 F 1 "R" H 7120 1855 50  0000 L CNN
-F 2 "" V 6980 1900 50  0001 C CNN
+F 2 "Resistor_THT:R_Axial_DIN0207_L6.3mm_D2.5mm_P10.16mm_Horizontal" V 6980 1900 50  0001 C CNN
 F 3 "~" H 7050 1900 50  0001 C CNN
 	1    7050 1900
@@
 F 0 "R22" V 6350 2450 50  0000 C CNN
 F 1 "500" V 6450 2500 50  0000 C CNN
-F 2 "" V 6380 2500 50  0001 C CNN
+F 2 "Resistor_THT:R_Axial_DIN0207_L6.3mm_D2.5mm_P10.16mm_Horizontal" V 6380 2500 50  0001 C CNN
 F 3 "~" H 6450 2500 50  0001 C CNN
 	1    6450 2500
@@
 F 0 "R24" H 6450 2500 50  0000 L CNN
 F 1 "10k" V 6600 2600 50  0000 L CNN
-F 2 "" V 6530 2650 50  0001 C CNN
+F 2 "Resistor_THT:R_Axial_DIN0207_L6.3mm_D2.5mm_P10.16mm_Horizontal" V 6530 2650 50  0001 C CNN
 F 3 "~" H 6600 2650 50  0001 C CNN
 	1    6600 2650
@@
 F 0 "J2" H 4150 1867 50  0000 C CNN
 F 1 "Conn_02x03_Top_Bottom" H 4150 1776 50  0000 C CNN
-F 2 "" H 4100 1550 50  0001 C CNN
+F 2 "Connector_PinSocket_2.54mm:PinSocket_2x03_P2.54mm_Vertical" H 4100 1550 50  0001 C CNN
 F 3 "~" H 4100 1550 50  0001 C CNN
 	1    4100 1550
@@
 F 0 "J3" H 4128 2776 50  0000 L CNN
 F 1 "Conn_01x02_Female" H 3600 2550 50  0000 L CNN
-F 2 "" H 4100 2800 50  0001 C CNN
+F 2 "Connector_PinSocket_2.54mm:PinSocket_1x02_P2.54mm_Vertical" H 4100 2800 50  0001 C CNN
 F 3 "~" H 4100 2800 50  0001 C CNN
 	1    4100 2800

Commit message: Made some progress on PCB layout. "Some" as in, kinda started.
Parts:
- J1: value Conn_01x03_Female -> RGB LED Connection
- J2: value Conn_02x03_Top_Bottom -> Switch Connections
- J3: value Conn_01x02_Female -> Battery Connection
- J4: value Conn_02x20_Top_Bottom -> LEDs on Buttons and Switches
- J5: value Conn_01x02_Female -> Motor Connection
Changed lines of the file:
@@
 P 3100 5050
 F 0 "J1" H 3128 5076 50  0000 L CNN
-F 1 "Conn_01x03_Female" H 2300 5300 50  0000 L CNN
+F 1 "RGB LED Connection" H 2300 5300 50  0000 L CNN
 F 2 "Connector_PinSocket_2.54mm:PinSocket_1x03_P2.54mm_Vertical" H 3100 5050 50  0001 C CNN
 F 3 "~" H 3100 5050 50  0001 C CNN
@@
 P 8900 1350
 F 0 "J5" H 8928 1326 50  0000 L CNN
-F 1 "Conn_01x02_Female" H 8500 1150 50  0000 L CNN
+F 1 "Motor Connection" H 8500 1150 50  0000 L CNN
 F 2 "Connector_PinSocket_2.54mm:PinSocket_1x02_P2.54mm_Vertical" H 8900 1350 50  0001 C CNN
 F 3 "~" H 8900 1350 50  0001 C CNN
@@
 P 6050 1450
 F 0 "J4" V 6146 2430 50  0000 L CNN
-F 1 "Conn_02x20_Top_Bottom" V 6450 950 50  0000 L CNN
+F 1 "LEDs on Buttons and Switches" V 6450 950 50  0000 L CNN
 F 2 "Connector_PinSocket_2.54mm:PinSocket_2x20_P2.54mm_Vertical" H 6050 1450 50  0001 C CNN
 F 3 "~" H 6050 1450 50  0001 C CNN
@@
 P 4100 1550
 F 0 "J2" H 4150 1867 50  0000 C CNN
-F 1 "Conn_02x03_Top_Bottom" H 4150 1776 50  0000 C CNN
+F 1 "Switch Connections" H 4150 1776 50  0000 C CNN
 F 2 "Connector_PinSocket_2.54mm:PinSocket_2x03_P2.54mm_Vertical" H 4100 1550 50  0001 C CNN
 F 3 "~" H 4100 1550 50  0001 C CNN
@@
 P 4100 2800
 F 0 "J3" H 4128 2776 50  0000 L CNN
-F 1 "Conn_01x02_Female" H 3600 2550 50  0000 L CNN
+F 1 "Battery Connection" H 3600 2550 50  0000 L CNN
 F 2 "Connector_PinSocket_2.54mm:PinSocket_1x02_P2.54mm_Vertical" H 4100 2800 50  0001 C CNN
 F 3 "~" H 4100 2800 50  0001 C CNN

Commit message: Layout mostly done, just need wires, copper areas, and edge cuts.
Parts:
- removed J2: Switch Connections, Connector_PinSocket_2.54mm:PinSocket_2x03_P2.54mm_Vertical, symbol Connector_Generic:Conn_02x03_Top_Bottom
- removed J4: LEDs on Buttons and Switches, Connector_PinSocket_2.54mm:PinSocket_2x20_P2.54mm_Vertical, symbol Connector_Generic:Conn_02x20_Top_Bottom
- added J2: Switches Connector, Connector_PinSocket_2.54mm:PinSocket_2x03_P2.54mm_Vertical, symbol Connector_Generic:Conn_02x03_Odd_Even
- added J4: LEDs on Buttons and Switches, Connector_PinSocket_2.54mm:PinSocket_2x20_P2.54mm_Vertical, symbol Connector_Generic:Conn_02x20_Odd_Even
Connections:
- net GND: now also J2.2 (Pin_2), J2.4 (Pin_4), J2.6 (Pin_6)
- net RGB_switch: now also J2.3 (Pin_3)
- net Reset: now also J2.1 (Pin_1)
- net VCC: now also J4.10 (Pin_10), J4.12 (Pin_12), J4.14 (Pin_14), J4.16 (Pin_16), J4.18 (Pin_18), J4.2 (Pin_2), J4.20 (Pin_20), J4.22 (Pin_22), J4.24 (Pin_24), J4.26 (Pin_26), J4.28 (Pin_28), J4.30 (Pin_30), J4.32 (Pin_32), J4.34 (Pin_34), J4.36 (Pin_36), J4.38 (Pin_38), J4.4 (Pin_4), J4.40 (Pin_40), J4.6 (Pin_6), J4.8 (Pin_8)
- net Vibrate_switch: now also J2.5 (Pin_5)
- net at R6.1: now also J4.1 (Pin_1)
- net at R19.1: now also J4.23 (Pin_23)
- net at R17.1: now also J4.19 (Pin_19)
- net at R18.1: now also J4.21 (Pin_21)
- net at R20.1: now also J4.25 (Pin_25)
- net at R21.1: now also J4.27 (Pin_27)
- net at R23.1: now also J4.29 (Pin_29)
- net at R25.1: now also J4.31 (Pin_31)
- net at R26.1: now also J4.33 (Pin_33)
- net at R27.1: now also J4.35 (Pin_35)
- net at R28.1: now also J4.37 (Pin_37)
- net at R7.1: now also J4.3 (Pin_3)
- net at R29.1: now also J4.39 (Pin_39)
- net at R9.1: now also J4.5 (Pin_5)
- net at R10.1: now also J4.7 (Pin_7)
- net at R12.1: now also J4.9 (Pin_9)
- net at R13.1: now also J4.11 (Pin_11)
- net at R14.1: now also J4.13 (Pin_13)
- net at R15.1: now also J4.15 (Pin_15)
- net at R16.1: now also J4.17 (Pin_17)
Changed lines of the file:
@@
 Connection ~ 8700 1650
-$Comp
-L Connector_Generic:Conn_02x20_Top_Bottom J4
-U 1 1 5FFF23C5
-P 6050 1450
-F 0 "J4" V 6146 2430 50  0000 L CNN
-F 1 "LEDs on Buttons and Switches" V 6450 950 50  0000 L CNN
-F 2 "Connector_PinSocket_2.54mm:PinSocket_2x20_P2.54mm_Vertical" H 6050 1450 50  0001 C CNN
-F 3 "~" H 6050 1450 50  0001 C CNN
-	1    6050 1450
-	0    -1   -1   0
-$EndComp
 $Comp
 L Device:R R7
@@
 	5150 1050 5150 1150
 Wire Wire Line
-	5150 1150 5250 1150
-Connection ~ 5150 1150
-Connection ~ 5250 1150
-Wire Wire Line
-	5250 1150 5350 1150
-Connection ~ 5350 1150
-Wire Wire Line
-	5350 1150 5450 1150
-Connection ~ 5450 1150
-Wire Wire Line
-	5450 1150 5550 1150
-Connection ~ 5550 1150
-Wire Wire Line
-	5550 1150 5650 1150
-Connection ~ 5650 1150
-Wire Wire Line
-	5650 1150 5750 1150
-Connection ~ 5750 1150
-Wire Wire Line
-	5750 1150 5850 1150
-Connection ~ 5850 1150
-Wire Wire Line
-	5850 1150 5950 1150
-Connection ~ 5950 1150
-Wire Wire Line
-	5950 1150 6050 1150
-Connection ~ 6050 1150
-Wire Wire Line
-	6050 1150 6150 1150
-Connection ~ 6150 1150
-Wire Wire Line
-	6150 1150 6250 1150
-Connection ~ 6250 1150
-Wire Wire Line
-	6250 1150 6350 1150
-Connection ~ 6350 1150
-Wire Wire Line
-	6350 1150 6450 1150
-Connection ~ 6450 1150
-Wire Wire Line
-	6450 1150 6550 1150
-Connection ~ 6550 1150
-Wire Wire Line
-	6550 1150 6650 1150
-Connection ~ 6650 1150
-Wire Wire Line
-	6650 1150 6750 1150
-Connection ~ 6750 1150
-Wire Wire Line
-	6750 1150 6850 1150
-Connection ~ 6850 1150
-Wire Wire Line
-	6850 1150 6950 1150
-Connection ~ 6950 1150
-Wire Wire Line
-	6950 1150 7050 1150
-Wire Wire Line
 	5150 1650 5150 1750
 Wire Wire Line
@@
 Wire Wire Line
 	7050 1750 7050 1650
-$Comp
-L Connector_Generic:Conn_02x03_Top_Bottom J2
-U 1 1 60082B98
-P 4100 1550
-F 0 "J2" H 4150 1867 50  0000 C CNN
-F 1 "Switch Connections" H 4150 1776 50  0000 C CNN
-F 2 "Connector_PinSocket_2.54mm:PinSocket_2x03_P2.54mm_Vertical" H 4100 1550 50  0001 C CNN
-F 3 "~" H 4100 1550 50  0001 C CNN
-	1    4100 1550
-	1    0    0    -1
-$EndComp
 $Comp
 L Connector:Conn_01x02_Female J3
@@
 Wire Notes Line
 	4450 2500 3550 2500
+Wire Wire Line
+	5150 1150 5250 1150
+$Comp
+L Connector_Generic:Conn_02x20_Odd_Even J4
+U 1 1 60001D64
+P 6050 1450
+F 0 "J4" V 6146 2429 50  0000 L CNN
+F 1 "LEDs on Buttons and Switches" V 6450 1100 50  0000 L CNN
+F 2 "Connector_PinSocket_2.54mm:PinSocket_2x20_P2.54mm_Vertical" H 6050 1450 50  0001 C CNN
+F 3 "~" H 6050 1450 50  0001 C CNN
+	1    6050 1450
+	0    -1   -1   0
+$EndComp
+Connection ~ 5150 1150
+Wire Wire Line
+	6950 1150 7050 1150
+Wire Wire Line
+	5250 1150 5350 1150
+Connection ~ 5250 1150
+Wire Wire Line
+	5350 1150 5450 1150
+Connection ~ 5350 1150
+Wire Wire Line
+	5450 1150 5550 1150
+Connection ~ 5450 1150
+Wire Wire Line
+	5650 1150 5550 1150
+Connection ~ 5550 1150
+Wire Wire Line
+	5650 1150 5750 1150
+Connection ~ 5650 1150
+Wire Wire Line
+	5750 1150 5850 1150
+Connection ~ 5750 1150
+Wire Wire Line
+	5850 1150 5950 1150
+Connection ~ 5850 1150
+Wire Wire Line
+	5950 1150 6050 1150
+Connection ~ 5950 1150
+Wire Wire Line
+	6050 1150 6150 1150
+Connection ~ 6050 1150
+Wire Wire Line
+	6150 1150 6250 1150
+Connection ~ 6150 1150
+Wire Wire Line
+	6250 1150 6350 1150
+Connection ~ 6250 1150
+Wire Wire Line
+	6350 1150 6450 1150
+Connection ~ 6350 1150
+Wire Wire Line
+	6450 1150 6550 1150
+Connection ~ 6450 1150
+Wire Wire Line
+	6550 1150 6650 1150
+Connection ~ 6550 1150
+Wire Wire Line
+	6650 1150 6750 1150
+Connection ~ 6650 1150
+Wire Wire Line
+	6750 1150 6850 1150
+Connection ~ 6750 1150
+Wire Wire Line
+	6850 1150 6950 1150
+Connection ~ 6850 1150
+Connection ~ 6950 1150
+$Comp
+L Connector_Generic:Conn_02x03_Odd_Even J2
+U 1 1 60045888
+P 4100 1550
+F 0 "J2" H 4150 1867 50  0000 C CNN
+F 1 "Switches Connector" H 4150 1776 50  0000 C CNN
+F 2 "Connector_PinSocket_2.54mm:PinSocket_2x03_P2.54mm_Vertical" H 4100 1550 50  0001 C CNN
+F 3 "~" H 4100 1550 50  0001 C CNN
+	1    4100 1550
+	1    0    0    -1
+$EndComp
 $EndSCHEMATC
