File: KarisGiftPCB/KarisGiftPCB.kicad_pcb (KiCad board)
At the start: 2 copper layers, 43 parts, among them J1 Conn_01x03_Female, J2 Conn_02x03_Top_Bottom, J3 Conn_01x02_Female, J4 Conn_02x20_Top_Bottom, J5 Conn_01x02_Female, Q1 2N3904, Q2 2N3906, Q3 2N3904, Q4 2N3904, Q5 2N3904, U1 ATtiny85V-10PU

Commit message: Made some progress on PCB layout. "Some" as in, kinda started.
Parts:
- J1: value Conn_01x03_Female -> RGB LED Connection
- J2: value Conn_02x03_Top_Bottom -> Switch Connections
- J3: value Conn_01x02_Female -> Battery Connection
- J4: value Conn_02x20_Top_Bottom -> LEDs on Buttons and Switches
- J5: value Conn_01x02_Female -> Motor Connection
- moved J3 111.7 mm to (47.0, 74.9), turned to 90 degrees
- moved J2 102.8 mm to (49.5, 108.0)
- moved U1 85.1 mm to (45.7, 83.8)
- moved Q2 73.4 mm to (139.7, 58.4)
- moved Q5 70.6 mm to (72.4, 55.9)
- moved D1 63.5 mm to (68.6, 133.3), turned to 180 degrees
- moved Q1 60.0 mm to (127.0, 58.4)
- moved Q4 57.8 mm to (110.5, 55.9)
- moved J1 57.2 mm to (61.0, 100.3)
- moved Q3 54.4 mm to (94.0, 57.1)
- moved J5 45.4 mm to (59.7, 119.4)
- moved R28 33.2 mm to (151.0, 77.7)
- moved R3 33.2 mm to (137.7, 77.7)
- moved R30 33.2 mm to (137.7, 81.8)
- moved R31 33.2 mm to (151.0, 81.8)
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
Commit message: Layout mostly done, just need wires, copper areas, and edge cuts.
Parts:
- J2: value Switch Connections -> Switches Connector
- moved R29 84.3 mm to (80.0, 77.5), turned to 270 degrees
- moved R21 82.4 mm to (95.2, 77.5), turned to 270 degrees
- moved R31 71.2 mm to (83.8, 105.4)
- moved R27 69.8 mm to (85.1, 77.5), turned to 270 degrees
- moved R28 68.5 mm to (82.5, 77.5), turned to 270 degrees
- moved R25 63.6 mm to (90.2, 77.5), turned to 270 degrees
- moved J4 58.4 mm to (128.3, 73.7), turned to 270 degrees
- moved R30 57.4 mm to (83.8, 101.6)
- moved R23 55.1 mm to (92.7, 77.5), turned to 270 degrees
- moved R1 55.1 mm to (118.1, 111.8)
- moved Q1 53.0 mm to (111.8, 109.2)
- moved R20 51.8 mm to (97.8, 77.5), turned to 270 degrees
- moved Q2 50.8 mm to (113.0, 101.6), turned to 270 degrees
- moved Q5 48.7 mm to (78.7, 104.1), turned to 270 degrees
- moved R24 48.3 mm to (92.7, 95.2)
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Connections:
- J2 pad 2: RGB_switch -> GND
- J2 pad 3: Vibrate_switch -> RGB_switch
- J2 pad 5: GND -> Vibrate_switch
- J4 pad 10: Net-(J4-Pad10) -> VCC
- J4 pad 12: Net-(J4-Pad12) -> VCC
- J4 pad 14: Net-(J4-Pad14) -> VCC
- J4 pad 16: Net-(J4-Pad16) -> VCC
- J4 pad 18: Net-(J4-Pad18) -> VCC
- J4 pad 2: Net-(J4-Pad2) -> VCC
- J4 pad 20: Net-(J4-Pad20) -> VCC
- J4 pad 21: VCC -> Net-(J4-Pad21)
- J4 pad 23: VCC -> Net-(J4-Pad23)
- J4 pad 25: VCC -> Net-(J4-Pad25)
- J4 pad 27: VCC -> Net-(J4-Pad27)
- J4 pad 29: VCC -> Net-(J4-Pad29)
- J4 pad 31: VCC -> Net-(J4-Pad31)
- J4 pad 33: VCC -> Net-(J4-Pad33)
- J4 pad 35: VCC -> Net-(J4-Pad35)
- J4 pad 37: VCC -> Net-(J4-Pad37)
- J4 pad 39: VCC -> Net-(J4-Pad39)
- J4 pad 4: Net-(J4-Pad4) -> VCC
- J4 pad 6: Net-(J4-Pad6) -> VCC
- J4 pad 8: Net-(J4-Pad8) -> VCC
- R10 pad 1: Net-(J4-Pad4) -> Net-(J4-Pad7)
- R12 pad 1: Net-(J4-Pad5) -> Net-(J4-Pad9)
- R13 pad 1: Net-(J4-Pad6) -> Net-(J4-Pad11)
- R14 pad 1: Net-(J4-Pad7) -> Net-(J4-Pad13)
- R15 pad 1: Net-(J4-Pad8) -> Net-(J4-Pad15)
- R16 pad 1: Net-(J4-Pad9) -> Net-(J4-Pad17)
- R17 pad 1: Net-(J4-Pad10) -> Net-(J4-Pad19)
- R18 pad 1: Net-(J4-Pad11) -> Net-(J4-Pad21)
- R19 pad 1: Net-(J4-Pad12) -> Net-(J4-Pad23)
- R20 pad 1: Net-(J4-Pad13) -> Net-(J4-Pad25)
- R21 pad 1: Net-(J4-Pad14) -> Net-(J4-Pad27)
- R23 pad 1: Net-(J4-Pad15) -> Net-(J4-Pad29)
- R25 pad 1: Net-(J4-Pad16) -> Net-(J4-Pad31)
- R26 pad 1: Net-(J4-Pad17) -> Net-(J4-Pad33)
- R27 pad 1: Net-(J4-Pad18) -> Net-(J4-Pad35)
- R28 pad 1: Net-(J4-Pad19) -> Net-(J4-Pad37)
- R29 pad 1: Net-(J4-Pad20) -> Net-(J4-Pad39)
- R7 pad 1: Net-(J4-Pad2) -> Net-(J4-Pad3)
- R9 pad 1: Net-(J4-Pad3) -> Net-(J4-Pad5)

Commit message: Finished board layout. Generated Gerber files.
Parts:
- Switches: renamed from J2; value Switches Connector -> Switches
- renumbered J5 to -Motor+, U1 to ATTiny85, J1 to RGB
Routing:
- net LED_cutoff: track 0.00 -> 82.3 mm
- net RGB_data: track 0.00 -> 37.8 mm
- net Vibrate_driver: track 0.00 -> 35.9 mm
- net Net-(Q3-Pad3): track 0.00 -> 26.7 mm
- net Net-(Q4-Pad3): track 0.00 -> 26.7 mm
- net Net-(D1-Pad2): track 0.00 -> 23.1 mm
- net Vibrate_switch: track 0.00 -> 19.4 mm
- net Reset: track 0.00 -> 18.9 mm
- net Net-(Q2-Pad2): track 0.00 -> 18.8 mm
- net RGB_switch: track 0.00 -> 15.8 mm
- net GND: track 0.00 -> 10.2 mm, vias 0 -> 2
- net Net-(Q1-Pad2): track 0.00 -> 9.97 mm
- net Net-(Q5-Pad2): track 0.00 -> 8.89 mm
- net Net-(Q4-Pad2): track 0.00 -> 8.67 mm
- net Net-(Q3-Pad2): track 0.00 -> 8.67 mm
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- added copper zone on B.Cu, net GND
- added copper zone on F.Cu, net VCC
Other:
- board outline added: 71.1 x 48.3 mm
- board text added: "- +"
- board text added: "Anode (+) Cathode (-)"
- board text added: "G D V"
- board text added: "Helpers: Mikayla, Lily, Malachi, Levi Leighton, Isaac, Aaron, Jacob"
- board text added: "Karis Gift V1.0 Zach English"
- board text added: "RGB"
- board text added: "Reset"
- board text added: "Vibrate"

Commit message: Updated names for correctness and spelling.
Other:
- board text added: "Helpers: Mikayla, Lily, Malachi, Levi Leighton, Isaac, Alex, Jakob"
- board text removed: "Helpers: Mikayla, Lily, Malachi, Levi Leighton, Isaac, Aaron, Jacob"
Changed lines of the file:
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@@
     (0 F.Cu signal)
     (31 B.Cu signal)
-    (32 B.Adhes user)
-    (33 F.Adhes user)
-    (34 B.Paste user)
-    (35 F.Paste user)
+    (32 B.Adhes user hide)
+    (33 F.Adhes user hide)
+    (34 B.Paste user hide)
+    (35 F.Paste user hide)
     (36 B.SilkS user)
     (37 F.SilkS user)
     (38 B.Mask user)
     (39 F.Mask user)
-    (40 Dwgs.User user)
-    (41 Cmts.User user)
-    (42 Eco1.User user)
-    (43 Eco2.User user)
+    (40 Dwgs.User user hide)
+    (41 Cmts.User user hide)
+    (42 Eco1.User user hide)
+    (43 Eco2.User user hide)
     (44 Edge.Cuts user)
-    (45 Margin user)
-    (46 B.CrtYd user)
-    (47 F.CrtYd user)
-    (48 B.Fab user)
+    (45 Margin user hide)
+    (46 B.CrtYd user hide)
+    (47 F.CrtYd user hide)
+    (48 B.Fab user hide)
     (49 F.Fab user hide)
   )
@@
     )
   )
-  (gr_text "Helpers: Mikayla, Lily, Malachi, Levi\nLeighton, Isaac, Aaron, Jacob" (at 102.87 82.55) (layer B.SilkS)
+  (gr_text "Helpers: Mikayla, Lily, Malachi, Levi\nLeighton, Isaac, Alex, Jakob" (at 102.87 82.55) (layer B.SilkS)
     (effects (font (size 1 1) (thickness 0.15)) (justify mirror))
   )

Commit message: Updated silkscreen and some code cleanup
Parts:
- added REF**: ZDE_Logo, KarisGiftPCB:ZDE_Logo, F.Cu at (73.4, 91.7)
Other:
- board text added: "Helpers: Kaya (Mikayla), Leely (Lily), Makai (Malachi), Wevi (Levi) Leeton (Leighton), Ithick (Isaac), Alik (Alex), Jayob (Jakob)"
- board text removed: "Helpers: Mikayla, Lily, Malachi, Levi Leighton, Isaac, Alex, Jakob"
Changed lines of the file:
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@@
     (tracks 105)
     (zones 0)
-    (modules 43)
+    (modules 44)
     (nets 40)
   )
@@
     (add_net Vibrate_switch)
   )
+  (module KarisGiftPCB:ZDE_Logo (layer F.Cu)
+    (at 73.406 91.694)
+    (fp_text reference REF** (at 0 0.5) (layer F.Fab)
+      (effects (font (size 1 1) (thickness 0.15)))
+    )
+    (fp_text value ZDE_Logo (at 0 -0.5) (layer F.Fab)
+      (effects (font (size 1 1) (thickness 0.15)))
+    )
+    (fp_arc (start 4.7498 5.715) (end 4.7244 3.8354) (angle -180) (layer F.SilkS) (width 0.25))
+    (fp_line (start 0 3.81) (end 7.62 3.81) (layer F.SilkS) (width 0.25))
+    (fp_line (start 7.62 0) (end 0 7.62) (layer F.SilkS) (width 0.25))
+    (fp_line (start 7.62 0) (end 0 0) (layer F.SilkS) (width 0.25))
+    (fp_line (start 7.62 7.62) (end 7.62 0) (layer F.SilkS) (width 0.25))
+    (fp_line (start 0 7.62) (end 7.62 7.62) (layer F.SilkS) (width 0.25))
+    (fp_line (start 0 5.08) (end 0 7.62) (layer F.SilkS) (width 0.25))
+    (fp_line (start 0 0) (end 0 5.08) (layer F.SilkS) (width 0.25))
+  )
   (module Connector_PinSocket_2.54mm:PinSocket_2x20_P2.54mm_Vertical (layer F.Cu)
     (at 128.27 73.66 270)
@@
     )
   )
-  (gr_text "Helpers: Mikayla, Lily, Malachi, Levi\nLeighton, Isaac, Alex, Jakob" (at 102.87 82.55) (layer B.SilkS)
+  (gr_text "Helpers: Kaya (Mikayla), Leely (Lily), Makai (Malachi), Wevi (Levi)\nLeeton (Leighton), Ithick (Isaac), Alik (Alex), Jayob (Jakob)" (at 102.87 82.55) (layer B.SilkS)
     (effects (font (size 1 1) (thickness 0.15)) (justify mirror))
   )
